Commit message: add a wheeled humanoid to the Gazebo office

File: simulation/models/robot/robot.urdf.xacro (robot description, xacro)
@@ -1,4 +1,17 @@
 <?xml version="1.0"?>
 <robot xmlns:xacro="http://www.ros.org/wiki/xacro" name="placecell_robot">
+  <material name="ceramic"><color rgba="0.9 0.93 0.95 1"/></material>
+  <material name="graphite"><color rgba="0.055 0.075 0.10 1"/></material>
+  <material name="cyan"><color rgba="0.04 0.8 0.94 1"/></material>
+  <material name="silver"><color rgba="0.42 0.50 0.56 1"/></material>
+  <material name="rubber"><color rgba="0.025 0.035 0.045 1"/></material>
+  <xacro:arg name="mesh_root" default="model://robot/meshes"/>
+  <xacro:property name="shell_mesh" value="$(arg mesh_root)/rounded_box.dae"/>
+  <xacro:macro name="shell" params="name xyz scale material rpy:='0 0 0'">
+    <visual name="${name}"><origin xyz="${xyz}" rpy="${rpy}"/>
+      <geometry><mesh filename="${shell_mesh}" scale="${scale}"/></geometry>
+      <material name="${material}"/>
+    </visual>
+  </xacro:macro>
   <xacro:macro name="inertia" params="mass xx yy zz">
     <inertial>
@@ -13,5 +26,7 @@
   <link name="base_link">
     <xacro:inertia mass="8" xx="0.11" yy="0.16" zz="0.23"/>
-    <visual><geometry><box size="0.48 0.34 0.16"/></geometry><material name="blue"><color rgba="0.08 0.3 0.65 1"/></material></visual>
+    <xacro:shell name="base_shell" xyz="0 0 0" scale="0.48 0.34 0.16" material="graphite"/>
+    <xacro:shell name="base_deck" xyz="0 0 0.064" scale="0.44 0.32 0.045" material="ceramic"/>
+    <xacro:shell name="front_light" xyz="0.237 0 0.005" scale="0.008 0.24 0.022" material="cyan"/>
     <collision><geometry><box size="0.48 0.34 0.16"/></geometry></collision>
   </link>
@@ -19,5 +34,7 @@
     <link name="${side}_wheel">
       <xacro:inertia mass="0.4" xx="0.0011" yy="0.002" zz="0.0011"/>
-      <visual><origin rpy="${pi/2} 0 0"/><geometry><cylinder radius="0.1" length="0.04"/></geometry><material name="rubber"><color rgba="0.08 0.08 0.08 1"/></material></visual>
+      <visual><origin rpy="${pi/2} 0 0"/><geometry><cylinder radius="0.1" length="0.04"/></geometry><material name="rubber"/></visual>
+      <visual name="hub"><origin xyz="0 ${0.022 if y > 0 else -0.022} 0" rpy="${pi/2} 0 0"/><geometry><cylinder radius="0.065" length="0.006"/></geometry><material name="silver"/></visual>
+      <visual name="hub_center"><origin xyz="0 ${0.026 if y > 0 else -0.026} 0" rpy="${pi/2} 0 0"/><geometry><cylinder radius="0.033" length="0.006"/></geometry><material name="cyan"/></visual>
       <collision><origin rpy="${pi/2} 0 0"/><geometry><cylinder radius="0.1" length="0.04"/></geometry></collision>
     </link>
@@ -41,6 +58,40 @@
   <xacro:caster name="front_caster" x="0.19"/>
   <xacro:caster name="rear_caster" x="-0.19"/>
+  <!-- The upper body is fixed; this robot navigates but does not manipulate objects. -->
+  <joint name="humanoid_joint" type="fixed">
+    <parent link="base_link"/><child link="humanoid_body"/><origin xyz="0 0 0.60"/>
+  </joint>
+  <link name="humanoid_body">
+    <xacro:inertia mass="2.0" xx="0.12" yy="0.12" zz="0.025"/>
+    <!-- All upper-body geometry fits the existing 0.48 x 0.46 m footprint. -->
+    <collision><origin xyz="-0.025 0 -0.025"/><geometry><box size="0.30 0.45 0.98"/></geometry></collision>
+    <!-- A narrow central column leaves the laser plane clear beyond its 8 cm near range. -->
+    <visual name="column"><origin xyz="0 0 -0.31"/><geometry><cylinder radius="0.033" length="0.42"/></geometry><material name="silver"/></visual>
+    <xacro:shell name="waist" xyz="-0.035 0 -0.10" scale="0.18 0.24 0.12" material="graphite"/>
+    <xacro:shell name="torso" xyz="-0.045 0 0.065" scale="0.20 0.29 0.29" material="ceramic"/>
+    <xacro:shell name="chest_screen" xyz="0.06 0 0.06" scale="0.016 0.16 0.15" material="graphite"/>
+    <xacro:shell name="chest_indicator" xyz="0.07 0 0.07" scale="0.006 0.10 0.012" material="cyan"/>
+    <xacro:shell name="chest_badge" xyz="0.07 0 0.025" scale="0.006 0.045 0.009" material="silver"/>
+    <visual name="neck"><origin xyz="0 0 0.25"/><geometry><cylinder radius="0.04" length="0.09"/></geometry><material name="graphite"/></visual>
+    <xacro:shell name="head" xyz="0.01 0 0.365" scale="0.20 0.24 0.20" material="ceramic"/>
+    <xacro:shell name="visor" xyz="0.108 0 0.365" scale="0.028 0.207 0.12" material="graphite"/>
+    <xacro:shell name="left_eye" xyz="0.125 0.053 0.378" scale="0.009 0.045 0.018" material="cyan"/>
+    <xacro:shell name="right_eye" xyz="0.125 -0.053 0.378" scale="0.009 0.045 0.018" material="cyan"/>
+    <xacro:macro name="arm" params="side sign">
+      <visual name="${side}_shoulder"><origin xyz="-0.045 ${sign*0.178} 0.15"/><geometry><sphere radius="0.047"/></geometry><material name="graphite"/></visual>
+      <xacro:shell name="${side}_upper_arm" xyz="-0.055 ${sign*0.184} 0.05" scale="0.085 0.070 0.18" material="ceramic"/>
+      <visual name="${side}_elbow"><origin xyz="-0.050 ${sign*0.184} -0.045"/><geometry><sphere radius="0.037"/></geometry><material name="graphite"/></visual>
+      <xacro:shell name="${side}_forearm" xyz="-0.014 ${sign*0.184} -0.12" rpy="0 -0.45 0" scale="0.074 0.070 0.16" material="ceramic"/>
+      <xacro:shell name="${side}_hand" xyz="0.028 ${sign*0.184} -0.20" scale="0.065 0.072 0.065" material="graphite"/>
+      <xacro:shell name="${side}_wrist_band" xyz="0.013 ${sign*0.184} -0.175" rpy="0 -0.45 0" scale="0.077 0.073 0.018" material="cyan"/>
+      <visual name="${side}_ear"><origin xyz="0.005 ${sign*0.125} 0.365" rpy="${pi/2} 0 0"/><geometry><cylinder radius="0.046" length="0.016"/></geometry><material name="cyan"/></visual>
+    </xacro:macro>
+    <xacro:arm side="left" sign="1"/>
+    <xacro:arm side="right" sign="-1"/>
+  </link>
   <link name="camera_link">
-    <visual><geometry><box size="0.04 0.12 0.04"/></geometry><material name="rubber"/></visual>
+    <xacro:shell name="depth_camera_housing" xyz="-0.025 0 0" scale="0.045 0.12 0.04" material="graphite"/>
+    <visual name="camera_mount"><origin xyz="-0.11 0 0"/><geometry><box size="0.22 0.025 0.025"/></geometry><material name="silver"/></visual>
+    <xacro:shell name="depth_camera_lens" xyz="0 0.037 0" scale="0.006 0.017 0.017" material="cyan"/>
   </link>
   <joint name="camera_joint" type="fixed"><parent link="base_link"/><child link="camera_link"/><origin xyz="0.22 0 0.35"/></joint>
